File: connectors.kicad_sch (KiCad schematic)
At the start: 13 parts, among them J1 RCJ-017, J2 USB4105-GF-A-120, J3 Conn_01x02_Pin, J4 Conn_01x02_Pin

Commit message: Replace 0201 diodes with recommended arrays and nothing (some were spurious and I think I don't need them)
Parts:
- removed D3, D4: PESD3V3Y1BSF, Diode_SMD:D_0201_0603Metric_Pad0.64x0.40mm_HandSolder, symbol Device:D_TVS
- added D5: PESD2USB3UVT-QR, Package_TO_SOT_SMD:SOT-23-3, symbol Power_Protection:ESDA5V3L
- D1: value PESD3V3Y1BSF -> CG0603MLU-3.3E; footprint Diode_SMD:D_0201_0603Metric_Pad0.64x0.40mm_HandSolder -> Diode_SMD:D_0603_1608Metric_Pad1.05x0.95mm_HandSolder; Mouser Part Number 771-PESD3V3Y1BSFYL -> 652-CG0603MLU-3.3E
Connections:
- net D+: now also D5.1 (K)
- net D-: now also D5.2 (K)
- net GND: now also D5.3 (A)
Changed lines of the file:
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@@
+	)
+	(junction
+		(at 106.68 95.25)
+		(diameter 0)
+		(color 0 0 0 0)
 	)
 	(junction
@@
 	)
 	(junction
-		(at 116.84 95.25)
-		(diameter 0)
-		(color 0 0 0 0)
-	)
-	(junction
 		(at 171.45 120.65)
 		(diameter 0)
@@
 	(wire
 		(pts
-			(xy 96.52 106.68) (xy 96.52 107.95)
+			(xy 104.14 110.49) (xy 104.14 111.76)
 		)
 		(stroke
@@
 	(wire
 		(pts
-			(xy 92.71 95.25) (xy 116.84 95.25)
+			(xy 92.71 95.25) (xy 106.68 95.25)
 		)
 		(stroke
@@
 	(wire
 		(pts
+			(xy 101.6 99.06) (xy 101.6 100.33)
+		)
+		(stroke
+			(width 0)
+			(type default)
+		)
+	)
+	(wire
+		(pts
 			(xy 92.71 97.79) (xy 96.52 97.79)
 		)
@@
 	(wire
 		(pts
-			(xy 116.84 95.25) (xy 119.38 95.25)
+			(xy 106.68 95.25) (xy 116.84 95.25)
 		)
 		(stroke
@@
 	(wire
 		(pts
-			(xy 116.84 106.68) (xy 116.84 107.95)
-		)
-		(stroke
-			(width 0)
-			(type default)
-		)
-	)
-	(wire
-		(pts
 			(xy 176.53 72.39) (xy 161.29 72.39)
 		)
@@
 	(wire
 		(pts
-			(xy 116.84 95.25) (xy 116.84 99.06)
-		)
-		(stroke
-			(width 0)
-			(type default)
-		)
-	)
-	(wire
-		(pts
 			(xy 171.45 133.35) (xy 172.72 133.35)
 		)
@@
 		(pts
 			(xy 167.64 102.87) (xy 171.45 102.87)
+		)
+		(stroke
+			(width 0)
+			(type default)
+		)
+	)
+	(wire
+		(pts
+			(xy 96.52 99.06) (xy 101.6 99.06)
+		)
+		(stroke
+			(width 0)
+			(type default)
+		)
+	)
+	(wire
+		(pts
+			(xy 106.68 95.25) (xy 106.68 100.33)
 		)
 		(stroke
@@
 	(text "Low C TVS for ESD protection"
 		(exclude_from_sim no)
-		(at 107.95 115.57 0)
+		(at 104.14 119.38 0)
 		(effects
 			(font
@@
 	(hierarchical_label "D-"
 		(shape bidirectional)
-		(at 119.38 95.25 0)
+		(at 116.84 95.25 0)
 		(fields_autoplaced yes)
 		(effects
@@
 	)
 	(symbol
-		(lib_id "power:GND")
-		(at 116.84 107.95 0)
-		(unit 1)
-		(exclude_from_sim no)
-		(in_bom yes)
-		(on_board yes)
-		(dnp no)
-		(fields_autoplaced yes)
-		(property "Reference" "#PWR07"
-			(at 116.84 114.3 0)
-			(effects
-				(font
-					(size 1.27 1.27)
-				)
-				(hide yes)
-			)
-		)
-		(property "Value" "GND"
-			(at 116.84 113.03 0)
-			(effects
-				(font
-					(size 1.27 1.27)
-				)
-			)
-		)
-		(property "Footprint" ""
-			(at 116.84 107.95 0)
-			(effects
-				(font
-					(size 1.27 1.27)
-				)
-				(hide yes)
-			)
-		)
-		(property "Datasheet" ""
-			(at 116.84 107.95 0)
-			(effects
-				(font
-					(size 1.27 1.27)
-				)
-				(hide yes)
-			)
-		)
-		(property "Description" "Power symbol creates a global label with name \"GND\" , ground"
-			(at 116.84 107.95 0)
-			(effects
-				(font
-					(size 1.27 1.27)
-				)
-				(hide yes)
-			)
-		)
-		(pin "1"
-		)
-		(instances
-			(project "BinauralMic"
-				(path "/d9e790b9-8aa4-4e58-8bd7-6ef4bc890627/ed99070c-0835-415c-8078-0f260c71dd6d"
-					(reference "#PWR07")
-					(unit 1)
-				)
-			)
-		)
-	)
-	(symbol
 		(lib_id "Connector:Conn_Coaxial")
 		(at 153.67 72.39 0)
@@
 	(symbol
 		(lib_id "power:GND")
-		(at 96.52 107.95 0)
+		(at 104.14 111.76 0)
 		(unit 1)
 		(exclude_from_sim no)
@@
 		(fields_autoplaced yes)
 		(property "Reference" "#PWR06"
-			(at 96.52 114.3 0)
+			(at 104.14 118.11 0)
 			(effects
 				(font
@@
 		)
 		(property "Value" "GND"
-			(at 96.52 113.03 0)
+			(at 104.14 116.84 0)
 			(effects
 				(font
@@
 		)
 		(property "Footprint" ""
-			(at 96.52 107.95 0)
+			(at 104.14 111.76 0)
 			(effects
 				(font
@@
 		)
 		(property "Datasheet" ""
-			(at 96.52 107.95 0)
+			(at 104.14 111.76 0)
 			(effects
 				(font
@@
 		)
 		(property "Description" "Power symbol creates a global label with name \"GND\" , ground"
-			(at 96.52 107.95 0)
+			(at 104.14 111.76 0)
 			(effects
 				(font
@@
 	)
 	(symbol
-		(lib_id "Device:D_TVS")
-		(at 116.84 102.87 90)
-		(unit 1)
-		(exclude_from_sim no)
-		(in_bom yes)
-		(on_board yes)
-		(dnp no)
-		(fields_autoplaced yes)
-		(property "Reference" "D4"
-			(at 119.38 101.5999 90)
-			(effects
-				(font
-					(size 1.27 1.27)
-				)
-				(justify right)
-			)
-		)
-		(property "Value" "PESD3V3Y1BSF"
-			(at 119.38 104.1399 90)
-			(effects
-				(font
-					(size 1.27 1.27)
-				)
-				(justify right)
-			)
-		)
-		(property "Footprint" "Diode_SMD:D_0201_0603Metric_Pad0.64x0.40mm_HandSolder"
-			(at 116.84 102.87 0)
-			(effects
-				(font
-					(size 1.27 1.27)
-				)
-				(hide yes)
-			)
-		)
-		(property "Datasheet" "https://www.mouser.com/datasheet/2/916/PESD3V3Y1BSF-1370637.pdf"
-			(at 116.84 102.87 0)
-			(effects
-				(font
-					(size 1.27 1.27)
-				)
-				(hide yes)
-			)
-		)
-		(property "Description" "Bidirectional transient-voltage-suppression diode"
-			(at 116.84 102.87 0)
-			(effects
-				(font
-					(size 1.27 1.27)
-				)
-				(hide yes)
-			)
-		)
-		(property "Mouser Part Number" "771-PESD3V3Y1BSFYL"
-			(at 116.84 102.87 0)
-			(effects
-				(font
-					(size 1.27 1.27)
-				)
-				(hide yes)
-			)
-		)
-		(pin "2"
-		)
-		(pin "1"
-		)
-		(instances
-			(project "BinauralMic"
-				(path "/d9e790b9-8aa4-4e58-8bd7-6ef4bc890627/ed99070c-0835-415c-8078-0f260c71dd6d"
-					(reference "D4")
-					(unit 1)
-				)
-			)
-		)
-	)
-	(symbol
 		(lib_id "Device:R")
 		(at 104.14 85.09 90)
@@
 	)
 	(symbol
-		(lib_id "Device:D_TVS")
-		(at 96.52 102.87 90)
+		(lib_id "Power_Protection:ESDA5V3L")
+		(at 104.14 105.41 0)
 		(unit 1)
 		(exclude_from_sim no)
@@
 		(dnp no)
 		(fields_autoplaced yes)
-		(property "Reference" "D3"
-			(at 99.06 101.5999 90)
-			(effects
-				(font
-					(size 1.27 1.27)
-				)
-				(justify right)
-			)
-		)
-		(property "Value" "PESD3V3Y1BSF"
-			(at 99.06 104.1399 90)
-			(effects
-				(font
-					(size 1.27 1.27)
-				)
-				(justify right)
-			)
-		)
-		(property "Footprint" "Diode_SMD:D_0201_0603Metric_Pad0.64x0.40mm_HandSolder"
-			(at 96.52 102.87 0)
-			(effects
-				(font
-					(size 1.27 1.27)
-				)
-				(hide yes)
-			)
-		)
-		(property "Datasheet" "https://www.mouser.com/datasheet/2/916/PESD3V3Y1BSF-1370637.pdf"
-			(at 96.52 102.87 0)
-			(effects
-				(font
-					(size 1.27 1.27)
-				)
-				(hide yes)
-			)
-		)
-		(property "Description" "Bidirectional transient-voltage-suppression diode"
-			(at 96.52 102.87 0)
-			(effects
-				(font
-					(size 1.27 1.27)
-				)
-				(hide yes)
-			)
-		)
-		(property "Mouser Part Number" "771-PESD3V3Y1BSFYL"
-			(at 96.52 102.87 0)
-			(effects
-				(font
-					(size 1.27 1.27)
-				)
-				(hide yes)
-			)
+		(property "Reference" "D5"
+			(at 110.49 104.1399 0)
+			(effects
+				(font
+					(size 1.27 1.27)
+				)
+				(justify left)
+			)
+		)
+		(property "Value" "PESD2USB3UVT-QR"
+			(at 110.49 106.6799 0)
+			(effects
+				(font
+					(size 1.27 1.27)
+				)
+				(justify left)
+			)
+		)
+		(property "Footprint" "Package_TO_SOT_SMD:SOT-23-3"
+			(at 88.9 115.57 0)
+			(effects
+				(font
+					(size 1.27 1.27)
+				)
+				(justify left)
+				(hide yes)
+			)
+		)
+		(property "Datasheet" "https://www.mouser.com/datasheet/2/916/PESD2USB3UVT_Q-3436360.pdf"
+			(at 104.14 120.65 0)
+			(effects
+				(font
+					(size 1.27 1.27)
+				)
+				(hide yes)
+			)
+		)
+		(property "Description" "TVS Diode Array, 2 Channels, SOT23"
+			(at 104.14 118.11 0)
+			(effects
+				(font
+					(size 1.27 1.27)
+				)
+				(hide yes)
+			)
+		)
+		(property "Mouser Part Number" "771-PESD2USB3UVT-QR"
+			(at 104.14 105.41 0)
+			(effects
+				(font
+					(size 1.27 1.27)
+				)
+				(hide yes)
+			)
+		)
+		(pin "1"
 		)
 		(pin "2"
 		)
-		(pin "1"
+		(pin "3"
 		)
 		(instances
 			(project ""
 				(path "/d9e790b9-8aa4-4e58-8bd7-6ef4bc890627/ed99070c-0835-415c-8078-0f260c71dd6d"
-					(reference "D3")
+					(reference "D5")
 					(unit 1)
 				)
@@
 			)
 		)
-		(property "Value" "PESD3V3Y1BSF"
+		(property "Value" "CG0603MLU-3.3E"
 			(at 163.83 78.7399 90)
 			(effects
@@
 			)
 		)
-		(property "Footprint" "Diode_SMD:D_0201_0603Metric_Pad0.64x0.40mm_HandSolder"
+		(property "Footprint" "Diode_SMD:D_0603_1608Metric_Pad1.05x0.95mm_HandSolder"
 			(at 161.29 77.47 0)
 			(effects
@@
 			)
 		)
-		(property "Datasheet" "https://www.mouser.com/datasheet/2/916/PESD3V3Y1BSF-1370637.pdf"
+		(property "Datasheet" "https://www.mouser.com/datasheet/2/54/MLU-778323.pdf"
 			(at 161.29 77.47 0)
 			(effects
@@
 			)
 		)
-		(property "Mouser Part Number" "771-PESD3V3Y1BSFYL"
+		(property "Mouser Part Number" "652-CG0603MLU-3.3E"
 			(at 161.29 77.47 0)
 			(effects
