File: ldo.kicad_sch (KiCad schematic)
At the start: 9 parts, among them U1 MIC5504-3.3YM5

Commit message: More layout, replaced chip crystal with a 2-pin oscillator
All is well with the world
Connections:
- net VDD renamed VCC_{A}
Changed lines of the file:
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@@
 		)
 	)
-	(hierarchical_label "VDD"
+	(hierarchical_label "VCC_{A}"
 		(shape output)
 		(at 180.34 96.52 90)

Commit message: Flipped inductor direction (dot towards EMI) and shuffled some components around
Hopefully a more rested me can fit this jigsaw a little better
Connections:
- net VCC: now also L2.1; no longer L2.2
- net VCC_{A}: now also L2.2; no longer L2.1
Other:
- moved on the sheet: L2
Changed lines of the file:
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@@
 	(symbol
 		(lib_id "Device:L")
-		(at 170.18 97.79 270)
-		(mirror x)
+		(at 170.18 97.79 90)
 		(unit 1)
 		(exclude_from_sim no)
